Commit message: Cpp script to patrol a square in the world

File: urdf/quad_f450_thermal.urdf (robot description, URDF)
Before this commit: robot quad_f450_thermal, 8 links, 7 joints
Links:
- added link /camera_quad_f450_monocular_link, mass 0.050075; collision box size=0.023813 0.027686 0.092682; visual mesh filename=package://uav_crowd_control/meshes/cam_link.STL
- link base_link_inertia: mass 1.65 -> 1.7
Joints:
- added joint /camera_quad_f450_monocular_joint: type fixed, parent base_link, child /camera_quad_f450_monocular_link, origin xyz=0.041421 -0.046913 -0.067515 rpy=0.0068235 0.7854 0
- joint /camera_quad_f450_thermal_joint: origin xyz=0 0 -0.013633 rpy=1.5708 1.5708 0 -> xyz=0.042355 0.046075 -0.066582 rpy=0.020785 0.7854 0
